File: Kicad/Hioki3540.sch (KiCad schematic (older format))
At the start: 118 parts, among them IC102 4051, IC105 MAX135, IC105 PGA204, IC108 AD822, IC109 OP177, IC111 AD620, IC114 LMC7660, IC115 LMC7660, IC116 AN7704, P103 INPUT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

Commit message: schematic: Add details of some cap values, R values, mark input diodes as schottky, polyfuse as a polyfuse, etc.
Parts:
- removed D105, D106, D107, D108: D, symbol D
- removed R133: R, symbol R
- added D105, D106, D107, D108: D_Schottky, symbol D_Schottky
- added R133: SMD100F-2018, symbol Polyfuse
- C144, C145: value CP -> 100u
- C151: value CP -> 330u
- C154: value CP -> 1000u
- IC107: renamed from U?; value REF19x -> REF193
- IC113: renamed from U?; value LTC1174 -> LTC1174-5
- IC114: value LMC7660 -> NJU7660AV; Alt (none) -> LMC7660
- L101: value INDUCTOR -> 100u
- R111: value R -> 49k9
- R112: value R -> 13k0
- R126: value R -> 10R0
- R127: value R -> 1k00
- R128: value R -> 100k
- R130, R131: value R -> 10k
- gave numbers to parts that had none: 1
Other:
- note added: "* Series inductor on all four lines\n(separate board)"
Changed lines of the file:
@@
 P 2800 3400
 F 0 "R131" V 2880 3400 50  0000 C CNN
-F 1 "R" V 2800 3400 50  0000 C CNN
+F 1 "10k" V 2800 3400 50  0000 C CNN
 F 2 "" V 2730 3400 30  0000 C CNN
 F 3 "" H 2800 3400 30  0000 C CNN
@@
 P 2800 3900
 F 0 "R130" V 2880 3900 50  0000 C CNN
-F 1 "R" V 2800 3900 50  0000 C CNN
+F 1 "10k" V 2800 3900 50  0000 C CNN
 F 2 "" V 2730 3900 30  0000 C CNN
 F 3 "" H 2800 3900 30  0000 C CNN
@@
 $EndComp
 $Comp
-L REF19x U?
+L REF19x IC107
 U 1 1 5611D6B9
 P 9500 11250
-F 0 "U?" H 9750 11500 60  0000 C CNN
-F 1 "REF19x" H 9800 10700 60  0000 C CNN
+F 0 "IC107" H 9750 11500 60  0000 C CNN
+F 1 "REF193" H 9800 10700 60  0000 C CNN
 F 2 "" H 9800 10700 60  0000 C CNN
 F 3 "" H 9800 10700 60  0000 C CNN
@@
 P 9950 6550
 F 0 "R126" V 10030 6550 50  0000 C CNN
-F 1 "R" V 9950 6550 50  0000 C CNN
+F 1 "10R0" V 9950 6550 50  0000 C CNN
 F 2 "" V 9880 6550 30  0000 C CNN
 F 3 "" H 9950 6550 30  0000 C CNN
@@
 P 11050 6550
 F 0 "R127" V 11130 6550 50  0000 C CNN
-F 1 "R" V 11050 6550 50  0000 C CNN
+F 1 "1k00" V 11050 6550 50  0000 C CNN
 F 2 "" V 10980 6550 30  0000 C CNN
 F 3 "" H 11050 6550 30  0000 C CNN
@@
 P 12200 6550
 F 0 "R128" V 12280 6550 50  0000 C CNN
-F 1 "R" V 12200 6550 50  0000 C CNN
+F 1 "100k" V 12200 6550 50  0000 C CNN
 F 2 "" V 12130 6550 30  0000 C CNN
 F 3 "" H 12200 6550 30  0000 C CNN
@@
 $EndComp
 $Comp
-L TD62004F U?
+L TD62004F IC112
 U 1 1 5616068E
 P 8350 8400
-F 0 "U?" H 8350 7850 60  0000 C CNN
+F 0 "IC112" H 8350 7850 60  0000 C CNN
 F 1 "TD62004F" H 8350 8950 60  0000 C CNN
 F 2 "" H 8350 8950 60  0000 C CNN
@@
 $EndComp
 $Comp
-L D D105
-U 1 1 561BBD5F
-P 2800 12650
-F 0 "D105" H 2800 12750 50  0000 C CNN
-F 1 "D" H 2800 12550 50  0000 C CNN
-F 2 "" H 2800 12650 60  0000 C CNN
-F 3 "" H 2800 12650 60  0000 C CNN
-	1    2800 12650
-	-1   0    0    1
-$EndComp
-$Comp
-L D D106
-U 1 1 561BC0AE
-P 3250 12650
-F 0 "D106" H 3250 12750 50  0000 C CNN
-F 1 "D" H 3250 12550 50  0000 C CNN
-F 2 "" H 3250 12650 60  0000 C CNN
-F 3 "" H 3250 12650 60  0000 C CNN
-	1    3250 12650
-	-1   0    0    1
-$EndComp
-$Comp
-L D D108
-U 1 1 561BC20E
-P 2800 12150
-F 0 "D108" H 2800 12250 50  0000 C CNN
-F 1 "D" H 2800 12050 50  0000 C CNN
-F 2 "" H 2800 12150 60  0000 C CNN
-F 3 "" H 2800 12150 60  0000 C CNN
-	1    2800 12150
-	-1   0    0    1
-$EndComp
-$Comp
-L D D107
-U 1 1 561BC214
-P 3250 12150
-F 0 "D107" H 3250 12250 50  0000 C CNN
-F 1 "D" H 3250 12050 50  0000 C CNN
-F 2 "" H 3250 12150 60  0000 C CNN
-F 3 "" H 3250 12150 60  0000 C CNN
-	1    3250 12150
-	-1   0    0    1
-$EndComp
-$Comp
 L CONN_01X02 P104
 U 1 1 561BC27C
@@
 Wire Wire Line
 	2550 12650 2650 12650
-$Comp
-L R R133
-U 1 1 561C1868
-P 5150 12400
-F 0 "R133" V 5230 12400 50  0000 C CNN
-F 1 "R" V 5150 12400 50  0000 C CNN
-F 2 "" V 5080 12400 30  0000 C CNN
-F 3 "" H 5150 12400 30  0000 C CNN
-	1    5150 12400
-	0    1    1    0
-$EndComp
 Wire Wire Line
 	4650 12400 4800 12400
@@
 	4800 12400 5000 12400
 $Comp
-L LTC1174 U?
+L LTC1174 IC113
 U 1 1 561C21BC
 P 6400 13000
-F 0 "U?" H 6550 13450 60  0000 C CNN
-F 1 "LTC1174" H 6700 12500 60  0000 C CNN
+F 0 "IC113" H 6550 13450 60  0000 C CNN
+F 1 "LTC1174-5" H 6700 12500 60  0000 C CNN
 F 2 "" H 6550 13450 60  0000 C CNN
 F 3 "" H 6550 13450 60  0000 C CNN
@@
 P 5500 12650
 F 0 "R111" V 5580 12650 50  0000 C CNN
-F 1 "R" V 5500 12650 50  0000 C CNN
+F 1 "49k9" V 5500 12650 50  0000 C CNN
 F 2 "" V 5430 12650 30  0000 C CNN
 F 3 "" H 5500 12650 30  0000 C CNN
@@
 P 5500 13150
 F 0 "R112" V 5580 13150 50  0000 C CNN
-F 1 "R" V 5500 13150 50  0000 C CNN
+F 1 "13k0" V 5500 13150 50  0000 C CNN
 F 2 "" V 5430 13150 30  0000 C CNN
 F 3 "" H 5500 13150 30  0000 C CNN
@@
 P 4800 12750
 F 0 "C154" H 4825 12850 50  0000 L CNN
-F 1 "CP" H 4825 12650 50  0000 L CNN
+F 1 "1000u" H 4825 12650 50  0000 L CNN
 F 2 "" H 4838 12600 30  0000 C CNN
 F 3 "" H 4800 12750 60  0000 C CNN
@@
 P 7600 13100
 F 0 "L101" V 7550 13100 50  0000 C CNN
-F 1 "INDUCTOR" V 7700 13100 50  0001 C CNN
+F 1 "100u" V 7450 13100 50  0000 C CNN
 F 2 "" H 7600 13100 60  0000 C CNN
 F 3 "" H 7600 13100 60  0000 C CNN
@@
 U 1 1 561C9908
 P 8000 13350
-F 0 "C151" H 8025 13450 50  0000 L CNN
-F 1 "CP" H 8025 13250 50  0000 L CNN
+F 0 "C151" H 7800 13500 50  0000 L CNN
+F 1 "330u" H 7800 13250 50  0000 L CNN
 F 2 "" H 8038 13200 30  0000 C CNN
 F 3 "" H 8000 13350 60  0000 C CNN
 	1    8000 13350
-	-1   0    0    1
+	1    0    0    -1
 $EndComp
 $Comp
@@
 U 1 1 561C9AC6
 P 8300 13350
-F 0 "C124" H 8325 13450 50  0000 L CNN
-F 1 "C" H 8325 13250 50  0000 L CNN
+F 0 "C124" H 8350 13250 50  0000 L CNN
+F 1 "C" H 8350 13450 50  0000 L CNN
 F 2 "" H 8338 13200 30  0000 C CNN
 F 3 "" H 8300 13350 60  0000 C CNN
@@
 P 9150 13700
 F 0 "IC114" H 9300 14200 60  0000 C CNN
-F 1 "LMC7660" H 9450 13200 60  0000 C CNN
+F 1 "NJU7660AV" H 9550 13200 60  0000 C CNN
 F 2 "" H 9300 14200 60  0000 C CNN
 F 3 "" H 9300 14200 60  0000 C CNN
+F 4 "LMC7660" H 9500 13100 60  0000 C CNN "Alt"
 	1    9150 13700
 	1    0    0    -1
@@
 U 1 1 561CEBE3
 P 8500 13950
-F 0 "C144" H 8525 14050 50  0000 L CNN
-F 1 "CP" H 8525 13850 50  0000 L CNN
+F 0 "C144" H 8300 14100 50  0000 L CNN
+F 1 "100u" H 8300 13850 50  0000 L CNN
 F 2 "" H 8538 13800 30  0000 C CNN
 F 3 "" H 8500 13950 60  0000 C CNN
 	1    8500 13950
-	-1   0    0    1
+	1    0    0    -1
 $EndComp
 Wire Wire Line
@@
 P 9900 13800
 F 0 "C145" H 9925 13900 50  0000 L CNN
-F 1 "CP" H 9925 13700 50  0000 L CNN
+F 1 "100u" H 9925 13700 50  0000 L CNN
 F 2 "" H 9938 13650 30  0000 C CNN
 F 3 "" H 9900 13800 60  0000 C CNN
@@
 Wire Wire Line
 	7100 6100 7100 6650
+$Comp
+L D_Schottky D108
+U 1 1 58C2822E
+P 2800 12150
+F 0 "D108" H 2800 12250 50  0000 C CNN
+F 1 "D_Schottky" H 2800 12050 50  0000 C CNN
+F 2 "" H 2800 12150 50  0000 C CNN
+F 3 "" H 2800 12150 50  0000 C CNN
+	1    2800 12150
+	-1   0    0    1
+$EndComp
+$Comp
+L D_Schottky D107
+U 1 1 58C28B87
+P 3250 12150
+F 0 "D107" H 3250 12250 50  0000 C CNN
+F 1 "D_Schottky" H 3250 12050 50  0000 C CNN
+F 2 "" H 3250 12150 50  0000 C CNN
+F 3 "" H 3250 12150 50  0000 C CNN
+	1    3250 12150
+	-1   0    0    1
+$EndComp
+$Comp
+L D_Schottky D105
+U 1 1 58C28F10
+P 2800 12650
+F 0 "D105" H 2800 12750 50  0000 C CNN
+F 1 "D_Schottky" H 2800 12550 50  0000 C CNN
+F 2 "" H 2800 12650 50  0000 C CNN
+F 3 "" H 2800 12650 50  0000 C CNN
+	1    2800 12650
+	-1   0    0    1
+$EndComp
+$Comp
+L D_Schottky D106
+U 1 1 58C290A6
+P 3250 12650
+F 0 "D106" H 3250 12750 50  0000 C CNN
+F 1 "D_Schottky" H 3250 12550 50  0000 C CNN
+F 2 "" H 3250 12650 50  0000 C CNN
+F 3 "" H 3250 12650 50  0000 C CNN
+	1    3250 12650
+	-1   0    0    1
+$EndComp
+Text Notes 650  4350 0    60   ~ 0
+* Series inductor on all four lines\n(separate board)
+$Comp
+L Polyfuse R133
+U 1 1 58C65635
+P 5150 12400
+F 0 "R133" V 5050 12400 50  0000 C CNN
+F 1 "SMD100F-2018" V 5350 12350 50  0000 C CNN
+F 2 "" H 5200 12200 50  0001 L CNN
+F 3 "" H 5150 12400 50  0001 C CNN
+F 4 "Litlefuse" V 5250 12350 60  0000 C CNN "Manufacturer"
+	1    5150 12400
+	0    1    1    0
+$EndComp
 $EndSCHEMATC

Commit message: Fix diode polarities in the analog section, add more resistor values, change some diodes to PN instead of Schottky.
Parts:
- removed Q102, Q103, Q104, Q105: J0, symbol D_Schottky_Small
- added Q102, Q103, Q104, Q105: J0, symbol D_Small
- R101, R107, R108: value R -> 49k9
- R109, R110: value R -> 1M00
- R118: value R -> 20k0
- R120: value R -> 10k0
- R129: value R -> 10k
Changed lines of the file:
@@
 P 2450 3600
 F 0 "R110" V 2530 3600 50  0000 C CNN
-F 1 "R" V 2450 3600 50  0000 C CNN
+F 1 "1M00" V 2450 3600 50  0000 C CNN
 F 2 "" V 2380 3600 30  0000 C CNN
 F 3 "" H 2450 3600 30  0000 C CNN
@@
 P 2450 4100
 F 0 "R109" V 2530 4100 50  0000 C CNN
-F 1 "R" V 2450 4100 50  0000 C CNN
+F 1 "1M00" V 2450 4100 50  0000 C CNN
 F 2 "" V 2380 4100 30  0000 C CNN
 F 3 "" H 2450 4100 30  0000 C CNN
@@
 $EndComp
 $Comp
-L D_Schottky_Small Q102
-U 1 1 5611A1A7
-P 3150 4100
-F 0 "Q102" H 3050 4200 50  0000 L CNN
-F 1 "J0" H 3100 4000 50  0000 L CNN
-F 2 "" V 3150 4100 60  0000 C CNN
-F 3 "" V 3150 4100 60  0000 C CNN
-	1    3150 4100
-	0    1    1    0
-$EndComp
-$Comp
-L D_Schottky_Small Q103
-U 1 1 5611A798
-P 3450 4100
-F 0 "Q103" H 3350 4200 50  0000 L CNN
-F 1 "J0" H 3400 4000 50  0000 L CNN
-F 2 "" V 3450 4100 60  0000 C CNN
-F 3 "" V 3450 4100 60  0000 C CNN
-	1    3450 4100
-	0    1    -1   0
-$EndComp
-$Comp
-L D_Schottky_Small Q104
-U 1 1 5611A7DD
-P 3150 3250
-F 0 "Q104" H 3050 3350 50  0000 L CNN
-F 1 "J0" H 3100 3150 50  0000 L CNN
-F 2 "" V 3150 3250 60  0000 C CNN
-F 3 "" V 3150 3250 60  0000 C CNN
-	1    3150 3250
-	0    1    -1   0
-$EndComp
-$Comp
-L D_Schottky_Small Q105
-U 1 1 5611A827
-P 3450 3250
-F 0 "Q105" H 3350 3350 50  0000 L CNN
-F 1 "J0" H 3400 3150 50  0000 L CNN
-F 2 "" V 3450 3250 60  0000 C CNN
-F 3 "" V 3450 3250 60  0000 C CNN
-	1    3450 3250
-	0    1    1    0
-$EndComp
-$Comp
 L PGA204 IC105
 U 1 1 5611B82F
@@
 F 3 "" H 3900 6800 60  0000 C CNN
 	1    3900 6800
-	0    -1   1    0
+	0    -1   -1   0
 $EndComp
 $Comp
@@
 F 3 "" H 4200 7550 60  0000 C CNN
 	1    4200 7550
-	-1   0    0    -1
+	1    0    0    -1
 $EndComp
 $Comp
@@
 P 3750 9050
 F 0 "R129" V 3830 9050 50  0000 C CNN
-F 1 "R" V 3750 9050 50  0000 C CNN
+F 1 "10k" V 3750 9050 50  0000 C CNN
 F 2 "" V 3680 9050 30  0000 C CNN
 F 3 "" H 3750 9050 30  0000 C CNN
@@
 P 7450 5850
 F 0 "R118" V 7530 5850 50  0000 C CNN
-F 1 "R" V 7450 5850 50  0000 C CNN
+F 1 "20k0" V 7450 5850 50  0000 C CNN
 F 2 "" V 7380 5850 30  0000 C CNN
 F 3 "" H 7450 5850 30  0000 C CNN
@@
 P 7450 6350
 F 0 "R120" V 7530 6350 50  0000 C CNN
-F 1 "R" V 7450 6350 50  0000 C CNN
+F 1 "10k0" V 7450 6350 50  0000 C CNN
 F 2 "" V 7380 6350 30  0000 C CNN
 F 3 "" H 7450 6350 30  0000 C CNN
@@
 P 5700 6750
 F 0 "R101" V 5780 6750 50  0000 C CNN
-F 1 "R" V 5700 6750 50  0000 C CNN
+F 1 "49k9" V 5700 6750 50  0000 C CNN
 F 2 "" V 5630 6750 30  0000 C CNN
 F 3 "" H 5700 6750 30  0000 C CNN
@@
 P 6200 8300
 F 0 "R107" V 6280 8300 50  0000 C CNN
-F 1 "R" V 6200 8300 50  0000 C CNN
+F 1 "49k9" V 6200 8300 50  0000 C CNN
 F 2 "" V 6130 8300 30  0000 C CNN
 F 3 "" H 6200 8300 30  0000 C CNN
@@
 P 6200 8800
 F 0 "R108" V 6280 8800 50  0000 C CNN
-F 1 "R" V 6200 8800 50  0000 C CNN
+F 1 "49k9" V 6200 8800 50  0000 C CNN
 F 2 "" V 6130 8800 30  0000 C CNN
 F 3 "" H 6200 8800 30  0000 C CNN
@@
 	0    1    1    0
 $EndComp
+$Comp
+L D_Small Q102
+U 1 1 58E23E71
+P 3150 4100
+F 0 "Q102" H 3100 4000 50  0000 L CNN
+F 1 "J0" H 3100 4200 50  0000 L CNN
+F 2 "" V 3150 4100 50  0000 C CNN
+F 3 "" V 3150 4100 50  0000 C CNN
+	1    3150 4100
+	0    1    -1   0
+$EndComp
+$Comp
+L D_Small Q103
+U 1 1 58E343E5
+P 3450 4100
+F 0 "Q103" H 3400 4000 50  0000 L CNN
+F 1 "J0" H 3400 4200 50  0000 L CNN
+F 2 "" V 3450 4100 50  0000 C CNN
+F 3 "" V 3450 4100 50  0000 C CNN
+	1    3450 4100
+	0    1    1    0
+$EndComp
+$Comp
+L D_Small Q105
+U 1 1 58E34770
+P 3450 3250
+F 0 "Q105" H 3400 3150 50  0000 L CNN
+F 1 "J0" H 3400 3350 50  0000 L CNN
+F 2 "" V 3450 3250 50  0000 C CNN
+F 3 "" V 3450 3250 50  0000 C CNN
+	1    3450 3250
+	0    1    1    0
+$EndComp
+$Comp
+L D_Small Q104
+U 1 1 58E34B07
+P 3150 3250
+F 0 "Q104" H 3100 3150 50  0000 L CNN
+F 1 "J0" H 3100 3350 50  0000 L CNN
+F 2 "" V 3150 3250 50  0000 C CNN
+F 3 "" V 3150 3250 50  0000 C CNN
+	1    3150 3250
+	0    1    -1   0
+$EndComp
 $EndSCHEMATC
